Commit message: System functions until pickposes, does calculate them but rotated incorrectly.
Currently a bit more broken due to a patch that doesn't work yet to
rotate the pose, and some weird path execution happening sometimes. In
general it does seem to operate as intended though, which is good.

File: src/abb_drivers/abb_ros2/robot_specific_config/abb_irb1200_support/urdf/irb1200_5_90.xacro (robot description, xacro)
@@ -3,5 +3,5 @@
   <xacro:arg name="use_fake_hardware" default="true"/>
   <xacro:property name="use_fake_hardware" value="$(arg use_fake_hardware)"/>
-  <xacro:arg name="rws_ip" default="192.168.125.1"/>
+  <xacro:arg name="rws_ip" default="192.168.125.12"/>
   <xacro:property name="rws_ip" value="$(arg rws_ip)"/>
   <xacro:arg name="rws_port" default="80"/>

File: src/abb_drivers/abb_ros2/robot_specific_config/abb_irb120_support/urdf/abb_irb120.urdf.xacro (robot description, xacro)
@@ -36,5 +36,5 @@
   <xacro:arg name="use_fake_hardware" default="true"/>
   <xacro:property name="use_fake_hardware" value="$(arg use_fake_hardware)"/> <!-- Not implemented, TODO. -->
-  <xacro:arg name="rws_ip" default="192.168.125.1"/>
+  <xacro:arg name="rws_ip" default="192.168.125.12"/>
   <xacro:property name="rws_ip" value="$(arg rws_ip)"/>
   <xacro:arg name="rws_port" default="80"/>
@@ -651,19 +651,19 @@
   <!-- Links & joints for tcp's. -->
   <link name="tool_tcp" />
-  <link name="camera_link" />
+  <link name="camera" />
   <link name="camera_tcp" />
-  <joint name="camera_link-link_5_joint" type="fixed">
+  <joint name="camera-link_5_joint" type="fixed">
     <origin xyz="0.125 0 0.06" rpy="0 0 0" />
     <parent link="link_5" />
-    <child link="camera_link" />
-  </joint>
-  <joint name="tool_tcp-flange_joint" type="fixed">
+    <child link="camera" />
+  </joint>
+  <joint name="tool_tcp-link_6_joint" type="fixed">
     <origin xyz="0.095 0 0" rpy="0 0 0" />
-    <parent link="flange" />
+    <parent link= "link_6" />
     <child link="tool_tcp" />
   </joint>
-  <joint name="camera_tcp-camera_link_joint" type="fixed">
+  <joint name="camera_tcp-camera_joint" type="fixed">
     <origin xyz="0 -0.0175 0" rpy="0 0 0" />
-    <parent link="camera_link" />
+    <parent link="camera" />
     <child link="camera_tcp" />
   </joint>
