Commit message: Updated sequences to now use 'correct' rotations.
The most important fixes made:
- Fixed camerapose positioning (again).
- Fixed pickpose generation through rotation of detected objects.
- Changed delay/timing in camera, not needed when the camera is
(essentially) static.

Found some issues:
- Planning for place positions.
- Path generation & execution order.
- System getting stuck in Pick poses due to single faulty
planning/execution error.
- Faulty/rather strange pointcloud positioning compared to actual input.
- Pilz planner has issues with LIN & CIRC planning.

File: src/abb_drivers/abb_ros2/robot_specific_config/abb_irb120_support/urdf/abb_irb120.urdf.xacro (robot description, xacro)
@@ -659,5 +659,5 @@
   </joint>
   <joint name="tool_tcp-link_6_joint" type="fixed">
-    <origin xyz="0.095 0 0" rpy="0 0 0" />
+    <origin xyz="0.095 0 0" rpy="0 -1.57079633 0" /> <!-- Rotation fix has been applied here, 90degree turn on the Y axis () -->
     <parent link= "link_6" />
     <child link="tool_tcp" />

Commit message: Functional Pickpose - Incorrect I/O control.
- Still has some issues with path planning & a unknown reason for
turning correct trajectories into incorrect, smoothed/optimized variants
that cause collisions with the crate that it detects, prints out and
then executes anyway.

- Also GPIO controller & Mitsubishi drivers are still present.

File: src/abb_drivers/abb_ros2/robot_specific_config/abb_irb120_support/urdf/abb_irb120.urdf.xacro (robot description, xacro)
@@ -552,5 +552,5 @@
               <mesh filename="package://abb_irb120_support/meshes/custom/crate_collision.stl"/>
           </geometry>
-          <origin rpy="0 0 0" xyz="0 0 0"/>
+          <origin rpy="0 0 0" xyz="0 0 -0.005"/> <!-- Minimal movement down to, the crate collision is slightly higher than the crate for collision-prevention. Slightly reduced due to small setup robotarm reach. -->
       </collision>
   </link>
@@ -573,22 +573,4 @@
   <!-- Add the crate inner bottom center link -->
   <link name="crate_inner_bottom_center"/>
-    <!-- <visual>
-      <geometry>
-        <box size="0.01 0.05 0.1"/>
-      </geometry>
-    </visual>
-  </link> -->
-  <!-- <link name="test_point_camerapose">
-    <visual>
-      <geometry>
-        <box size="0.4 0.4 0.2"/>
-      </geometry>
-    </visual>
-  </link>
-  <joint name="test_joint" type="fixed">
-      <parent link="world"/>
-      <child link="test_point_camerapose"/>
-      <origin rpy="1.6 0 0" xyz="0.310 0 0.322"/>
-  </joint> -->
   <joint name="crate_joint" type="fixed">
       <parent link="robot_stand"/>
@@ -668,3 +650,16 @@
     <child link="camera_tcp" />
   </joint>
+<!-- Link and joint for Place center (See abb_irb120_params.yaml in StateMachine). -->
+  <link name="place_center" />
+  <joint name="place_center-world" type="fixed">
+    <origin xyz="0.3 -0.42 0" rpy="0 0 0" />
+    <parent link="world" />
+    <child link="place_center" />
+  </joint>
+  <link name="example" />
+  <joint name="example-world" type="fixed">
+    <origin xyz="0.29 -0.43 0.009250" rpy="3.1415842 0 1.5707963" />
+    <parent link="world" />
+    <child link="example" />
+  </joint>
 </robot>

File: src/mitsubishi_driver/melfa_description/urdf/rv5as_custom/rv5as.urdf (robot description, URDF)
Before this commit: robot rv5as, 17 links, 16 joints
Links:
- added link Test_Position_Place
Joints:
- added joint joink: type fixed, parent world, child Test_Position_Place, origin xyz=-0.25 0.25 -0.008 rpy=0 0 0

Commit message: Cleaned up some code, slightly changed URDF to fix a slight mismatch in camera output not lining up with the crate.

File: src/abb_drivers/abb_ros2/robot_specific_config/abb_irb120_support/urdf/abb_irb120.urdf.xacro (robot description, xacro)
@@ -582,5 +582,5 @@
       <parent link="crate"/>
       <child link="crate_foam"/>
-      <origin rpy="0 0 0" xyz="0 0 0"/>
+      <origin rpy="0 0 0" xyz="0 0 -0.003"/>
   </joint>
   <!-- Add the joint to connect the crate_inner_bottom_center to crate -->
